Commit message: second_commit

File: my_robot_description/urdf/mobile_base.xacro (robot description, xacro)
@@ -25,5 +25,5 @@
             <origin xyz="0 0 0" rpy="0 0 0" />
             <geometry>
-                <mesh filename="package://my_robot_description/meshes/autobot/base_link.STL" />
+                <mesh filename="package://my_robot_description/meshes/autobot/base_link.stl" />
             </geometry>
             <material name="${blue_material}" />
@@ -32,5 +32,5 @@
             <origin xyz="0 0 0" rpy="0 0 0" />
             <geometry>
-                <mesh filename="package://my_robot_description/meshes/autobot/base_link.STL" />
+                <mesh filename="package://my_robot_description/meshes/autobot/base_link.stl" />
             </geometry>
         </collision>
@@ -57,5 +57,5 @@
             <origin xyz="0 0 0" rpy="0 0 0" />
             <geometry>
-                <mesh filename="package://my_robot_description/meshes/autobot/right_wheel.STL" />
+                <mesh filename="package://my_robot_description/meshes/autobot/right_wheel.stl" />
             </geometry>
             <material name="${black_material}" />
@@ -64,5 +64,5 @@
             <origin xyz="0 0 0" rpy="0 0 0" />
             <geometry>
-                <mesh filename="package://my_robot_description/meshes/autobot/right_wheel.STL" />
+                <mesh filename="package://my_robot_description/meshes/autobot/right_wheel.stl" />
             </geometry>
         </collision>
@@ -92,5 +92,5 @@
             <origin xyz="0 0 0" rpy="0 0 0" />
             <geometry>
-                <mesh filename="package://my_robot_description/meshes/autobot/left_wheel.STL" />
+                <mesh filename="package://my_robot_description/meshes/autobot/left_wheel.stl" />
             </geometry>
             <material name="${black_material}" />
@@ -99,5 +99,5 @@
             <origin xyz="0 0 0" rpy="0 0 0" />
             <geometry>
-                <mesh filename="package://my_robot_description/meshes/autobot/left_wheel.STL" />
+                <mesh filename="package://my_robot_description/meshes/autobot/left_wheel.stl" />
             </geometry>
         </collision>
@@ -127,5 +127,5 @@
             <origin xyz="0 0 0" rpy="0 0 0" />
             <geometry>
-                <mesh filename="package://my_robot_description/meshes/autobot/front_wheel.STL" />
+                <mesh filename="package://my_robot_description/meshes/autobot/front_wheel.stl" />
             </geometry>
             <material name="${black_material}" />
@@ -134,5 +134,5 @@
             <origin xyz="0 0 0" rpy="0 0 0" />
             <geometry>
-                <mesh filename="package://my_robot_description/meshes/autobot/front_wheel.STL" />
+                <mesh filename="package://my_robot_description/meshes/autobot/front_wheel.stl" />
             </geometry>
         </collision>
